File: Lithium/lithium.brd (EAGLE design)
At the start: 90.2 x 81.6 mm, 67 parts, among them J3 PJ-040X, Q1 J112, Q10 VP3203, Q2 J112, Q3 ZTX694B, Q4 ZVN4306A, Q5 ZVN4306A, Q6 J112, Q7 J112, Q8 ZVN4306A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

Commit message: Li-ion powered version WIP
Changed lines of the file:
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@@
 <contactref element="J6" pad="1"/>
 <contactref element="J10" pad="1"/>
-<wire x1="46.99" y1="59.69" x2="52.07" y2="53.34" width="0" layer="19" extent="1-1"/>
+<via x="20.32" y="36.83" extent="1-16" drill="0.5"/>
+<via x="13.97" y="54.61" extent="1-16" drill="0.5"/>
+<via x="10.16" y="50.8" extent="1-16" drill="0.5"/>
+<via x="10.16" y="46.99" extent="1-16" drill="0.5"/>
+<via x="13.97" y="46.99" extent="1-16" drill="0.5"/>
+<via x="12.7" y="35.56" extent="1-16" drill="0.5"/>
+<via x="2.54" y="40.64" extent="1-16" drill="0.5"/>
+<via x="29.21" y="38.1" extent="1-16" drill="0.5"/>
+<via x="38.1" y="38.1" extent="1-16" drill="0.5"/>
+<via x="45.72" y="39.37" extent="1-16" drill="0.5"/>
+<via x="44.45" y="46.99" extent="1-16" drill="0.5"/>
+<via x="49.53" y="45.72" extent="1-16" drill="0.5"/>
+<via x="33.02" y="49.53" extent="1-16" drill="0.5"/>
+<via x="29.21" y="46.99" extent="1-16" drill="0.5"/>
+<via x="31.75" y="54.61" extent="1-16" drill="0.5"/>
+<via x="53.975" y="52.07" extent="1-16" drill="0.5"/>
+<via x="57.15" y="53.34" extent="1-16" drill="0.5"/>
+<via x="59.69" y="46.99" extent="1-16" drill="0.5"/>
+<via x="78.74" y="45.72" extent="1-16" drill="0.5"/>
+<via x="78.74" y="43.18" extent="1-16" drill="0.5"/>
+<via x="73.66" y="49.53" extent="1-16" drill="0.5"/>
+<via x="73.66" y="53.34" extent="1-16" drill="0.5"/>
+<via x="64.77" y="38.1" extent="1-16" drill="0.5"/>
+<via x="59.69" y="39.37" extent="1-16" drill="0.5"/>
+<via x="57.15" y="36.83" extent="1-16" drill="0.5"/>
+<via x="68.58" y="33.02" extent="1-16" drill="0.5"/>
+<via x="73.66" y="33.02" extent="1-16" drill="0.5"/>
+<via x="86.36" y="35.56" extent="1-16" drill="0.5"/>
+<via x="87.63" y="44.45" extent="1-16" drill="0.5"/>
+<via x="66.04" y="50.8" extent="1-16" drill="0.5"/>
+<via x="6.35" y="63.5" extent="1-16" drill="0.5"/>
+<via x="5.08" y="78.74" extent="1-16" drill="0.5"/>
+<via x="15.24" y="74.93" extent="1-16" drill="0.5"/>
+<via x="3.81" y="72.39" extent="1-16" drill="0.5"/>
+<via x="24.13" y="74.93" extent="1-16" drill="0.5"/>
+<via x="27.94" y="80.01" extent="1-16" drill="0.5"/>
+<via x="40.64" y="78.74" extent="1-16" drill="0.5"/>
+<via x="49.53" y="78.74" extent="1-16" drill="0.5"/>
+<via x="34.29" y="73.66" extent="1-16" drill="0.5"/>
+<via x="34.29" y="67.31" extent="1-16" drill="0.5"/>
+<via x="37.465" y="70.485" extent="1-16" drill="0.5"/>
+<via x="41.91" y="64.77" extent="1-16" drill="0.5"/>
+<via x="50.8" y="62.23" extent="1-16" drill="0.5"/>
+<via x="52.705" y="69.85" extent="1-16" drill="0.5"/>
+<via x="46.99" y="63.5" extent="1-16" drill="0.5"/>
+<via x="45.4025" y="67.945" extent="1-16" drill="0.5"/>
+<via x="24.13" y="60.96" extent="1-16" drill="0.5"/>
+<via x="19.05" y="62.23" extent="1-16" drill="0.5"/>
+<via x="19.05" y="68.58" extent="1-16" drill="0.5"/>
+<via x="13.97" y="68.58" extent="1-16" drill="0.5"/>
+<via x="19.05" y="45.72" extent="1-16" drill="0.5"/>
+<via x="20.32" y="50.165" extent="1-16" drill="0.5"/>
+<via x="32.385" y="43.18" extent="1-16" drill="0.5"/>
+<via x="48.895" y="32.385" extent="1-16" drill="0.5"/>
+<via x="50.8" y="36.83" extent="1-16" drill="0.5"/>
+<via x="55.245" y="46.99" extent="1-16" drill="0.5"/>
+<via x="54.9275" y="49.8475" extent="1-16" drill="0.5"/>
+<wire x1="29.845" y1="59.69" x2="31.75" y2="54.61" width="0" layer="19" extent="1-1"/>
 </signal>
 <signal name="N$6">

Commit message: Stamp holes removed
Parts:
- added J12: (no value), SparkFun-Connectors:1X02
- added LOGO1: LOGO-MANTIS, my:LOGO-MANTIS
- moved C8 53.8 mm to (46.4, 26.0)
- moved J9 53.8 mm to (27.3, 27.9)
- moved Q8 53.8 mm to (64.5, 21.0)
- moved C10 53.8 mm to (48.3, 8.89)
- moved C9 53.8 mm to (36.2, 25.4)
- moved D3 53.8 mm to (43.2, 8.89)
- moved J11 53.8 mm to (62.5, 7.62)
- moved J4 53.8 mm to (40.0, 20.3)
- moved Q7 53.8 mm to (26.0, 8.89)
- moved R17 53.8 mm to (34.9, 15.2)
- moved R21 53.8 mm to (34.9, 7.62)
- moved R24 53.8 mm to (47.6, 15.2)
- moved J6 53.8 mm to (62.5, 17.8)
- moved Q6 53.8 mm to (26.0, 12.7)
- moved Q9 53.8 mm to (64.5, 14.6)
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Connections:
- net GND: now also J12.1
- net VBAT: now also J12.2
Routing:
- net VBAT: track 0.00 -> 11.1 mm
Other:
- board size 90.2 x 81.6 mm -> 90.2 x 55.6 mm
- board text added: "Portuum Lithium"
