File: 2PCBs/tin_of_fets.sch (EAGLE design)
At the start: 59 parts, among them J4 PJ-040X, Q1 J112, Q2 J112, Q3 ZVN4306A, Q4 ZVN4306A, Q5 ZTX694B, Q6 J112, Q7 J112, Q8 ZVN4306A, Q9 ZVN4306A

Commit message: Small improvements
Parts:
- removed J11, J6: (no value), SparkFun-Connectors:M01PTH
- added D5: 1N4148, SparkFun-DiscreteSemi:DIODE1N4148
- D2, D3: value (none) -> 1N5819-B; device SparkFun-DiscreteSemi:DIODEPTH -> diode:1N5819-B
Connections:
- net +12V: now also D5.C
- net GND: no longer J11.1, J6.1
- net N$23: now also D5.A
