File: Statuum/statuum.brd (EAGLE design)
At the start: 104.1 x 91.4 mm, 75 parts, among them IC1 LM317MABT, J1 POWER_JACKPTH, J2 NRJ3HF-1, J3 RCJ-21XXMILL, Q1 2N5484, Q10 IRF510, Q2 2N5484, Q3 IRF510, Q4 IRF510, Q5 BD140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

Commit message: Small fix
Parts:
- C3: device SparkFun-Capacitors:CPOL-RADIAL-1000UF-63V -> my-cap:CPOL-RADIAL-16/7.5
- C9: value 47uF/35V -> 47uF/63V
- D10, D3, D4, D9: value BLUE -> YELLOW
- Q1, Q2, Q7, Q8: value 2N5484 -> PN4393
- R20, R21, R4, R5: value 820 -> 560
- R22, R6: value 4.7k -> 5.1k
Changed lines of the file:
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@@
 <attribute name="VALUE" x="38.227" y="69.215" size="0.8128" layer="27" ratio="20" rot="R270"/>
 </element>
-<element name="D3" library="my" package="LED3MM-SM" value="BLUE" x="15.24" y="58.42" smashed="yes" rot="R180">
+<element name="D3" library="my" package="LED3MM-SM" value="YELLOW" x="15.24" y="58.42" smashed="yes" rot="R180">
 <attribute name="NAME" x="13.335" y="59.944" size="0.8128" layer="25" ratio="20" rot="R180"/>
 <attribute name="VALUE" x="13.335" y="60.071" size="0.8128" layer="27" ratio="20" rot="R180"/>
 </element>
-<element name="D4" library="my" package="LED3MM-SM" value="BLUE" x="7.62" y="58.42" smashed="yes" rot="R180">
+<element name="D4" library="my" package="LED3MM-SM" value="YELLOW" x="7.62" y="58.42" smashed="yes" rot="R180">
 <attribute name="NAME" x="5.715" y="59.944" size="0.8128" layer="25" ratio="20" rot="R180"/>
 <attribute name="VALUE" x="5.715" y="60.071" size="0.8128" layer="27" ratio="20" rot="R180"/>
 </element>
-<element name="D9" library="my" package="LED3MM-SM" value="BLUE" x="52.07" y="58.42" smashed="yes">
+<element name="D9" library="my" package="LED3MM-SM" value="YELLOW" x="52.07" y="58.42" smashed="yes">
 <attribute name="NAME" x="54.61" y="58.166" size="0.8128" layer="25" ratio="20"/>
 <attribute name="VALUE" x="53.975" y="56.769" size="0.8128" layer="27" ratio="20"/>
 </element>
-<element name="D10" library="my" package="LED3MM-SM" value="BLUE" x="59.69" y="58.42" smashed="yes">
+<element name="D10" library="my" package="LED3MM-SM" value="YELLOW" x="59.69" y="58.42" smashed="yes">
 <attribute name="NAME" x="62.23" y="58.166" size="0.8128" layer="25" ratio="20"/>
 <attribute name="VALUE" x="61.595" y="56.769" size="0.8128" layer="27" ratio="20"/>
 </element>
-<element name="Q1" library="my-tran" package="TO-92" value="2N5484" x="17.78" y="67.31" smashed="yes" rot="R270">
+<element name="Q1" library="my-tran" package="TO-92" value="PN4393" x="17.78" y="67.31" smashed="yes" rot="R270">
 <attribute name="NAME" x="14.605" y="67.945" size="0.8128" layer="25" ratio="20" rot="R270"/>
 <attribute name="VALUE" x="16.51" y="64.135" size="0.8128" layer="27" ratio="20" rot="R270"/>
 </element>
-<element name="Q2" library="my-tran" package="TO-92" value="2N5484" x="11.43" y="67.31" smashed="yes" rot="R90">
+<element name="Q2" library="my-tran" package="TO-92" value="PN4393" x="11.43" y="67.31" smashed="yes" rot="R90">
 <attribute name="NAME" x="8.255" y="66.675" size="0.8128" layer="25" ratio="20" rot="R90"/>
 <attribute name="VALUE" x="12.7" y="70.485" size="0.8128" layer="27" ratio="20" rot="R90"/>
 </element>
-<element name="Q7" library="my-tran" package="TO-92" value="2N5484" x="49.53" y="67.31" smashed="yes" rot="R90">
+<element name="Q7" library="my-tran" package="TO-92" value="PN4393" x="49.53" y="67.31" smashed="yes" rot="R90">
 <attribute name="NAME" x="46.355" y="66.675" size="0.8128" layer="25" ratio="20" rot="R90"/>
 <attribute name="VALUE" x="50.8" y="70.485" size="0.8128" layer="27" ratio="20" rot="R90"/>
 </element>
-<element name="Q8" library="my-tran" package="TO-92" value="2N5484" x="55.88" y="67.31" smashed="yes" rot="R270">
+<element name="Q8" library="my-tran" package="TO-92" value="PN4393" x="55.88" y="67.31" smashed="yes" rot="R270">
 <attribute name="NAME" x="59.69" y="67.945" size="0.8128" layer="25" ratio="20" rot="R270"/>
 <attribute name="VALUE" x="54.61" y="64.135" size="0.8128" layer="27" ratio="20" rot="R270"/>
@@
 <attribute name="VALUE" x="5.969" y="44.196" size="0.8128" layer="27" font="vector" ratio="20" rot="R270"/>
 </element>
-<element name="R20" library="my-res" package="AXIAL-0.4" value="820" x="41.91" y="62.23" smashed="yes" rot="R180">
+<element name="R20" library="my-res" package="AXIAL-0.4" value="560" x="41.91" y="62.23" smashed="yes" rot="R180">
 <attribute name="NAME" x="36.83" y="64.135" size="0.8128" layer="25" font="vector" ratio="20"/>
 <attribute name="VALUE" x="44.196" y="62.611" size="0.8128" layer="27" font="vector" ratio="20" rot="R180"/>
 </element>
-<element name="R21" library="my-res" package="AXIAL-0.4" value="820" x="55.88" y="62.23" smashed="yes" rot="R180">
+<element name="R21" library="my-res" package="AXIAL-0.4" value="560" x="55.88" y="62.23" smashed="yes" rot="R180">
 <attribute name="NAME" x="52.705" y="64.135" size="0.8128" layer="25" font="vector" ratio="20"/>
 <attribute name="VALUE" x="58.166" y="62.611" size="0.8128" layer="27" font="vector" ratio="20" rot="R180"/>
@@
 <attribute name="VALUE" x="53.594" y="54.229" size="0.8128" layer="27" font="vector" ratio="20"/>
 </element>
-<element name="R22" library="my-res" package="AXIAL-0.4" value="4.7k" x="41.91" y="58.42" smashed="yes" rot="R180">
+<element name="R22" library="my-res" package="AXIAL-0.4" value="5.1k" x="41.91" y="58.42" smashed="yes" rot="R180">
 <attribute name="NAME" x="36.83" y="59.69" size="0.8128" layer="25" font="vector" ratio="20"/>
 <attribute name="VALUE" x="44.196" y="58.801" size="0.8128" layer="27" font="vector" ratio="20" rot="R180"/>
@@
 <attribute name="VALUE" x="13.716" y="76.581" size="0.8128" layer="27" font="vector" ratio="20" rot="R180"/>
 </element>
-<element name="R4" library="my-res" package="AXIAL-0.4" value="820" x="25.4" y="62.23" smashed="yes">
+<element name="R4" library="my-res" package="AXIAL-0.4" value="560" x="25.4" y="62.23" smashed="yes">
 <attribute name="NAME" x="20.955" y="63.5" size="0.8128" layer="25" font="vector" ratio="20"/>
 <attribute name="VALUE" x="23.114" y="61.849" size="0.8128" layer="27" font="vector" ratio="20"/>
 </element>
-<element name="R5" library="my-res" package="AXIAL-0.4" value="820" x="11.43" y="62.23" smashed="yes">
+<element name="R5" library="my-res" package="AXIAL-0.4" value="560" x="11.43" y="62.23" smashed="yes">
 <attribute name="NAME" x="8.255" y="64.135" size="0.8128" layer="25" font="vector" ratio="20"/>
 <attribute name="VALUE" x="9.144" y="61.849" size="0.8128" layer="27" font="vector" ratio="20"/>
 </element>
-<element name="R6" library="my-res" package="AXIAL-0.4" value="4.7k" x="25.4" y="58.42" smashed="yes">
+<element name="R6" library="my-res" package="AXIAL-0.4" value="5.1k" x="25.4" y="58.42" smashed="yes">
 <attribute name="NAME" x="20.955" y="59.69" size="0.8128" layer="25" font="vector" ratio="20"/>
 <attribute name="VALUE" x="23.114" y="58.039" size="0.8128" layer="27" font="vector" ratio="20"/>
@@
 <attribute name="VALUE" x="92.202" y="85.471" size="1.016" layer="21" ratio="12" rot="R270"/>
 </element>
-<element name="C3" library="SparkFun-Capacitors" package="CPOL-RADIAL-1000UF-63V" value="4700uF/35V" x="76.2" y="62.23" smashed="yes">
+<element name="C3" library="my-cap" package="CPOL-RADIAL-16/7.5" value="4700uF/35V" x="76.2" y="62.23" smashed="yes">
 <attribute name="VALUE" x="73.66" y="71.12" size="0.8128" layer="27" ratio="20"/>
 <attribute name="NAME" x="74.93" y="67.31" size="0.8128" layer="25" ratio="20"/>
@@
 <attribute name="VALUE" x="82.55" y="48.895" size="0.8128" layer="27" ratio="20" rot="R90"/>
 </element>
-<element name="C9" library="my-cap" package="CPOL-RADIAL-6.5/2.5" value="47uF/35V" x="71.12" y="45.72" smashed="yes" rot="R90">
+<element name="C9" library="my-cap" package="CPOL-RADIAL-6.5/2.5" value="47uF/63V" x="71.12" y="45.72" smashed="yes" rot="R90">
 <attribute name="VALUE" x="75.438" y="43.815" size="0.8128" layer="27" ratio="20" rot="R90"/>
 <attribute name="NAME" x="69.469" y="44.958" size="0.8128" layer="25" ratio="20" rot="R90"/>

Commit message: Small fix
Parts:
- R19, R3: value 100k -> 1.2k
Changed lines of the file:
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@@
 <attribute name="VALUE" x="58.166" y="72.771" size="0.8128" layer="27" font="vector" ratio="20" rot="R180"/>
 </element>
-<element name="R19" library="my-res" package="AXIAL-0.4" value="100k" x="55.88" y="76.2" smashed="yes">
+<element name="R19" library="my-res" package="AXIAL-0.4" value="1.2k" x="55.88" y="76.2" smashed="yes">
 <attribute name="NAME" x="52.705" y="78.105" size="0.8128" layer="25" font="vector" ratio="20"/>
 <attribute name="VALUE" x="53.594" y="75.819" size="0.8128" layer="27" font="vector" ratio="20"/>
@@
 <attribute name="VALUE" x="44.196" y="58.801" size="0.8128" layer="27" font="vector" ratio="20" rot="R180"/>
 </element>
-<element name="R3" library="my-res" package="AXIAL-0.4" value="100k" x="11.43" y="76.2" smashed="yes" rot="R180">
+<element name="R3" library="my-res" package="AXIAL-0.4" value="1.2k" x="11.43" y="76.2" smashed="yes" rot="R180">
 <attribute name="NAME" x="8.255" y="78.105" size="0.8128" layer="25" font="vector" ratio="20"/>
 <attribute name="VALUE" x="13.716" y="76.581" size="0.8128" layer="27" font="vector" ratio="20" rot="R180"/>
