File: Statuum/statuum.sch (EAGLE design)
At the start: 75 parts, among them IC1 LM317MABT, J1 POWER_JACKPTH, J2 NRJ3HF-1, J3 RCJ-21XXMILL, Q1 2N5484, Q10 IRF510, Q2 2N5484, Q3 IRF510, Q4 IRF510, Q5 BD140, Q6 BC547, Q7 2N5484, Q8 2N5484, Q9 IRF510

Commit message: Small fix
Parts:
- C3: device SparkFun-Capacitors:CAP_POLPTH3 -> my-cap:CAP_POLPTH-16/7.5
- C9: value 47uF/35V -> 47uF/63V
- D10, D3, D4, D9: value BLUE -> YELLOW
- Q1, Q2, Q7, Q8: value 2N5484 -> PN4393; device my-tran:2N5484 -> my-tran:PN4393
- R20, R21, R4, R5: value 820 -> 560
- R22, R6: value 4.7k -> 5.1k
Other:
- note added: "4.7V"
Changed lines of the file:
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@@
 <parts>
 <part name="C7" library="my-cap" deviceset="CAP_POL" device="PTH-8/3.5" value="470u"/>
-<part name="Q1" library="my-tran" deviceset="2N5484" device="" value="2N5484"/>
-<part name="Q2" library="my-tran" deviceset="2N5484" device="" value="2N5484"/>
-<part name="R4" library="my-res" deviceset="RESISTOR" device="PTH-1/4W" value="820"/>
-<part name="R5" library="my-res" deviceset="RESISTOR" device="PTH-1/4W" value="820"/>
+<part name="Q1" library="my-tran" deviceset="PN4393" device="" value="PN4393"/>
+<part name="Q2" library="my-tran" deviceset="PN4393" device="" value="PN4393"/>
+<part name="R4" library="my-res" deviceset="RESISTOR" device="PTH-1/4W" value="560"/>
+<part name="R5" library="my-res" deviceset="RESISTOR" device="PTH-1/4W" value="560"/>
 <part name="GND4" library="SparkFun-Aesthetics" deviceset="GND" device=""/>
 <part name="R1" library="my-res" deviceset="RESISTOR" device="PTH-1/4W" value="680"/>
@@
 <part name="SUPPLY4" library="SparkFun-Aesthetics" deviceset="VCC" device=""/>
 <part name="R7" library="my-res" deviceset="RESISTOR" device="PTH-1/4W" value="1Meg"/>
-<part name="D3" library="my" deviceset="LED" device="3MM-SM" value="BLUE"/>
-<part name="R6" library="my-res" deviceset="RESISTOR" device="PTH-1/4W" value="4.7k"/>
+<part name="D3" library="my" deviceset="LED" device="3MM-SM" value="YELLOW"/>
+<part name="R6" library="my-res" deviceset="RESISTOR" device="PTH-1/4W" value="5.1k"/>
 <part name="GND5" library="SparkFun-Aesthetics" deviceset="GND" device=""/>
 <part name="SUPPLY3" library="SparkFun-Aesthetics" deviceset="VCC" device=""/>
@@
 <part name="GND1" library="SparkFun-Aesthetics" deviceset="GND" device=""/>
 <part name="SUPPLY1" library="SparkFun-Aesthetics" deviceset="VCC" device=""/>
-<part name="D4" library="my" deviceset="LED" device="3MM-SM" value="BLUE"/>
+<part name="D4" library="my" deviceset="LED" device="3MM-SM" value="YELLOW"/>
 <part name="C8" library="my-cap" deviceset="CAP_POL" device="PTH-8/3.5" value="470u"/>
 <part name="C17" library="my-cap" deviceset="CAP_POL" device="PTH-8/3.5" value="470u"/>
-<part name="Q7" library="my-tran" deviceset="2N5484" device="" value="2N5484"/>
-<part name="Q8" library="my-tran" deviceset="2N5484" device="" value="2N5484"/>
-<part name="R20" library="my-res" deviceset="RESISTOR" device="PTH-1/4W" value="820"/>
-<part name="R21" library="my-res" deviceset="RESISTOR" device="PTH-1/4W" value="820"/>
+<part name="Q7" library="my-tran" deviceset="PN4393" device="" value="PN4393"/>
+<part name="Q8" library="my-tran" deviceset="PN4393" device="" value="PN4393"/>
+<part name="R20" library="my-res" deviceset="RESISTOR" device="PTH-1/4W" value="560"/>
+<part name="R21" library="my-res" deviceset="RESISTOR" device="PTH-1/4W" value="560"/>
 <part name="GND14" library="SparkFun-Aesthetics" deviceset="GND" device=""/>
 <part name="R17" library="my-res" deviceset="RESISTOR" device="PTH-1/4W" value="680"/>
@@
 <part name="SUPPLY10" library="SparkFun-Aesthetics" deviceset="VCC" device=""/>
 <part name="R23" library="my-res" deviceset="RESISTOR" device="PTH-1/4W" value="1Meg"/>
-<part name="D9" library="my" deviceset="LED" device="3MM-SM" value="BLUE"/>
-<part name="R22" library="my-res" deviceset="RESISTOR" device="PTH-1/4W" value="4.7k"/>
+<part name="D9" library="my" deviceset="LED" device="3MM-SM" value="YELLOW"/>
+<part name="R22" library="my-res" deviceset="RESISTOR" device="PTH-1/4W" value="5.1k"/>
 <part name="GND15" library="SparkFun-Aesthetics" deviceset="GND" device=""/>
 <part name="SUPPLY9" library="SparkFun-Aesthetics" deviceset="VCC" device=""/>
@@
 <part name="GND12" library="SparkFun-Aesthetics" deviceset="GND" device=""/>
 <part name="SUPPLY6" library="SparkFun-Aesthetics" deviceset="VCC" device=""/>
-<part name="D10" library="my" deviceset="LED" device="3MM-SM" value="BLUE"/>
+<part name="D10" library="my" deviceset="LED" device="3MM-SM" value="YELLOW"/>
 <part name="C18" library="my-cap" deviceset="CAP_POL" device="PTH-8/3.5" value="470u"/>
 <part name="J3" library="my" deviceset="RCJ-21XX" device="MILL"/>
@@
 <part name="D6" library="SparkFun-DiscreteSemi" deviceset="DIODE" device="PTH"/>
 <part name="GND3" library="SparkFun-Aesthetics" deviceset="GND" device=""/>
-<part name="C3" library="SparkFun-Capacitors" deviceset="CAP_POL" device="PTH3" value="4700uF/35V"/>
+<part name="C3" library="my-cap" deviceset="CAP_POL" device="PTH-16/7.5" value="4700uF/35V"/>
 <part name="C4" library="my-cap" deviceset="CAP_POL" device="PTH-16/7.5" value="4700uF/35V"/>
 <part name="GND6" library="SparkFun-Aesthetics" deviceset="GND" device=""/>
@@
 <part name="Q5" library="transistor-pnp" deviceset="BD140" device=""/>
 <part name="Q6" library="my-tran" deviceset="BC547" device=""/>
-<part name="C9" library="my-cap" deviceset="CAP_POL" device="PTH-6.5/2.5" value="47uF/35V"/>
+<part name="C9" library="my-cap" deviceset="CAP_POL" device="PTH-6.5/2.5" value="47uF/63V"/>
 <part name="GND9" library="SparkFun-Aesthetics" deviceset="GND" device=""/>
 <part name="C5" library="SparkFun-Capacitors" deviceset="CAP" device="PTH" value="1uF"/>
@@
 <text x="254" y="149.86" size="1.778" layer="97" rot="R90">Optionally Zener</text>
 <text x="215.9" y="83.82" size="1.778" layer="97">+15V</text>
+<text x="55.88" y="180.34" size="1.778" layer="97">4.7V</text>
+<text x="236.22" y="180.34" size="1.778" layer="97">4.7V</text>
 </plain>
 <instances>

Commit message: Small fix
Parts:
- R19, R3: value 100k -> 1.2k
Changed lines of the file:
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@@
 <part name="R1" library="my-res" deviceset="RESISTOR" device="PTH-1/4W" value="680"/>
 <part name="R2" library="my-res" deviceset="RESISTOR" device="PTH-1/4W" value="3.3k"/>
-<part name="R3" library="my-res" deviceset="RESISTOR" device="PTH-1/4W" value="100k"/>
+<part name="R3" library="my-res" deviceset="RESISTOR" device="PTH-1/4W" value="1.2k"/>
 <part name="GND2" library="SparkFun-Aesthetics" deviceset="GND" device=""/>
 <part name="SUPPLY2" library="SparkFun-Aesthetics" deviceset="VCC" device=""/>
@@
 <part name="R17" library="my-res" deviceset="RESISTOR" device="PTH-1/4W" value="680"/>
 <part name="R18" library="my-res" deviceset="RESISTOR" device="PTH-1/4W" value="3.3k"/>
-<part name="R19" library="my-res" deviceset="RESISTOR" device="PTH-1/4W" value="100k"/>
+<part name="R19" library="my-res" deviceset="RESISTOR" device="PTH-1/4W" value="1.2k"/>
 <part name="GND13" library="SparkFun-Aesthetics" deviceset="GND" device=""/>
 <part name="SUPPLY8" library="SparkFun-Aesthetics" deviceset="VCC" device=""/>
